File: controller/Adafruit HUZZAH32 ESP32 Feather.kicad_sch (KiCad schematic)
At the start: 34 parts, among them IC1 CP2104, Q1 mmbt2222, Q2 mmbt2222, Q3 DMG3415U, SW2 KMR2, U2 AP2112-3.3, U3 MCP73831T-2ACI/OT, X1 JSTPH, X4 20329

Commit message: fixed connecgtio
Parts:
- U?: footprint Adafruit HUZZAH32 ESP32 Feather:WROOM32_SKINNY -> ESP32-WROOM-32:ESP32­WROOM­32E_EXP
Connections:
- net 3.3V: now also U?.2 (3V3)
- net A0_DAC2: now also U?.11 (IO26)
- net A13_I35: now also U?.7 (IO35)
- net A1_DAC1: now also U?.10 (IO25)
- net A2_I34: now also U?.6 (IO34)
- net A5_IO4: now also U?.26 (IO4)
- net GND: now also U?.1 (GND), U?.38 (GND), U?.39 (GND), U?.40 (GND), U?.41 (GND), U?.42 (GND), U?.43 (GND), U?.44 (GND), U?.45 (GND), U?.46 (GND), U?.47 (GND)
- net GPIO0: now also U?.25 (IO0)
- net GPIO2: now also U?.24 (IO2)
- net IO12_A11: now also U?.14 (IO12)
- net IO13_A12: now also U?.16 (IO13)
- net IO14_A6: now also U?.13 (IO14)
- net IO15_A8: now also U?.23 (IO15)
- net IO16: now also U?.27 (IO16)
- net IO17: now also U?.28 (IO17)
- net IO21: now also U?.33 (IO21)
- net IO27_A10: now also U?.12 (IO27)
- net IO32_A7: now also U?.8 (IO32)
- net IO33_A9: now also U?.9 (IO33)
- net MISO: now also U?.31 (IO19)
- net MOSI: now also U?.30 (IO18)
- net SCK: now also U?.29 (IO5)
- net SCL: now also U?.36 (IO22)
- net SDA: now also U?.37 (IO23)
